Commit message: improve urdf all commits from joint-control

File: march_ws/src/march_description/urdf/march-iii.xacro (robot description, xacro)
@@ -117,7 +117,8 @@
     <link name="upper_leg_left">
         <visual>
-            <origin xyz="0 0 ${-upper_leg_height/2}" rpy="0 0 0"/>
-            <geometry>
-                <box size="${width} ${width} ${upper_leg_height}"/>
+            <origin xyz="0 0 ${-0.9*upper_leg_height}" rpy="0 0 1.8"/>
+            <geometry>
+<!--                <box size="${width} ${width} ${upper_leg_height}"/>-->
+                <mesh filename="package://march_description/urdf/stl-files/UpperLegRight1.stl" scale="1.2 1.2 1.2"/>
             </geometry>
         </visual>
@@ -134,7 +135,8 @@
     <link name="lower_leg_left">
         <visual>
-            <origin xyz="0 0 ${-lower_leg_height/2}" rpy="0 0 0"/>
-            <geometry>
-                <box size="${width} ${width} ${lower_leg_height}"/>
+            <origin xyz="${-0.4*width} 0 ${-1.0*lower_leg_height}" rpy="0 0 1.8"/>
+            <geometry>
+<!--                <box size="${width} ${width} ${lower_leg_height}"/>-->
+                <mesh filename="package://march_description/urdf/stl-files/LowerLeg.stl" scale="1.2 1.2 1.2"/>
             </geometry>
         </visual>
@@ -173,7 +175,8 @@
     <link name="upper_leg_right">
         <visual>
-            <origin xyz="0 0 ${-upper_leg_height/2}" rpy="0 0 0"/>
-            <geometry>
-                <box size="${width} ${width} ${upper_leg_height}"/>
+            <origin xyz="0 0 ${-0.9*upper_leg_height}" rpy="0 0 -1.8"/>
+            <geometry>
+<!--                <box size="${width} ${width} ${upper_leg_height}"/>-->
+                <mesh filename="package://march_description/urdf/stl-files/UpperLegRight1.stl" scale="1.2 1.2 1.2"/>
             </geometry>
         </visual>

Commit message: change lengths to the right lengths displayed in catia

File: march_ws/src/march_description/urdf/march-iii.xacro (robot description, xacro)
@@ -11,11 +11,11 @@
     <xacro:property name="mass" value="1"/> <!-- arbitrary value for mass -->
     <xacro:property name="width" value="0.05"/> <!-- Square dimensions (widthxwidth) of beams -->
-    <xacro:property name="upper_leg_height" value="${0.39}"/>
+    <xacro:property name="upper_leg_height" value="${0.385}"/>
     <xacro:property name="upper_leg_mass" value="1.080"/>
-    <xacro:property name="lower_leg_height" value="${0.39}"/>
+    <xacro:property name="lower_leg_height" value="${0.385}"/>
     <xacro:property name="lower_leg_mass" value="1.133"/>
-    <xacro:property name="foot_height" value="${0.14*1}"/>
+    <xacro:property name="foot_height" value="${0.184}"/>
     <xacro:property name="foot_mass" value="0.393"/>
-    <xacro:property name="hip_height" value="0.33"/>
+    <xacro:property name="hip_height" value="0.420"/>
     <xacro:property name="hip_rotation_lower_limit" value="${-15*pi/180}"/> <!-- rad -->
     <xacro:property name="hip_rotation_upper_limit" value="${105*pi/180}"/> <!-- rad -->
@@ -137,6 +137,6 @@
             <origin xyz="${-0.4*width} 0 ${-1.0*lower_leg_height}" rpy="0 0 1.8"/>
             <geometry>
-<!--                <box size="${width} ${width} ${lower_leg_height}"/>-->
-                <mesh filename="package://march_description/urdf/stl-files/LowerLeg.stl" scale="1.2 1.2 1.2"/>
+                <box size="${width} ${width} ${lower_leg_height}"/>
+<!--                <mesh filename="package://march_description/urdf/stl-files/LowerLeg.stl" scale="1.2 1.2 1.2"/>-->
             </geometry>
         </visual>

Commit message: Adjust position, velocity and effort limits

File: march_ws/src/march_description/urdf/march-iii.xacro (robot description, xacro)
@@ -20,14 +20,14 @@
     <xacro:property name="hip_rotation_lower_limit" value="${-15*pi/180}"/> <!-- rad -->
     <xacro:property name="hip_rotation_upper_limit" value="${105*pi/180}"/> <!-- rad -->
-    <xacro:property name="hip_effort_limit" value="1000.0"/> <!-- Rad -->
-    <xacro:property name="hip_velocity_limit" value="1000.0"/> <!-- rad/s -->
-    <xacro:property name="knee_rotation_lower_limit" value="${-15*pi/180}"/>
-    <xacro:property name="knee_rotation_upper_limit" value="${105*pi/180}"/>
-    <xacro:property name="knee_effort_limit" value="1000.0"/>
-    <xacro:property name="knee_velocity_limit" value="1000.0"/>
+    <xacro:property name="hip_effort_limit" value="10927.0"/> <!-- IU -->
+    <xacro:property name="hip_velocity_limit" value="48.0"/> <!-- rad/s -->
+    <xacro:property name="knee_rotation_lower_limit" value="${-5*pi/180}"/>
+    <xacro:property name="knee_rotation_upper_limit" value="${115*pi/180}"/>
+    <xacro:property name="knee_effort_limit" value="10927.0"/>
+    <xacro:property name="knee_velocity_limit" value="48.0"/>
     <xacro:property name="ankle_rotation_lower_limit" value="${-15*pi/180}"/>
-    <xacro:property name="ankle_rotation_upper_limit" value="${20*pi/180}"/>
-    <xacro:property name="ankle_effort_limit" value="1000.0"/>
-    <xacro:property name="ankle_velocity_limit" value="1000.0"/>
+    <xacro:property name="ankle_rotation_upper_limit" value="${30*pi/180}"/>
+    <xacro:property name="ankle_effort_limit" value="10927.0"/>
+    <xacro:property name="ankle_velocity_limit" value="15.0"/>
     <xacro:property name="hover_height" value="0.3"/>
     <xacro:property name="camera_link" value="0.05"/> <!-- Size of square 'camera' box -->

Commit message: Add HAA without angle in frame. Add joint state publisher in launch file

File: march_ws/src/march_description/urdf/march-iii.xacro (robot description, xacro)
@@ -18,8 +18,14 @@
     <xacro:property name="foot_mass" value="0.393"/>
     <xacro:property name="hip_height" value="0.420"/>
-    <xacro:property name="hip_rotation_lower_limit" value="${-15*pi/180}"/> <!-- rad -->
-    <xacro:property name="hip_rotation_upper_limit" value="${105*pi/180}"/> <!-- rad -->
-    <xacro:property name="hip_effort_limit" value="10927.0"/> <!-- IU -->
-    <xacro:property name="hip_velocity_limit" value="48.0"/> <!-- rad/s -->
+    <xacro:property name="hip_base_height" value="0.160"/>
+    <xacro:property name="hip_moving_height" value="0.130"/>
+    <xacro:property name="hipFE_rotation_lower_limit" value="${-15*pi/180}"/> <!-- rad -->
+    <xacro:property name="hipFE_rotation_upper_limit" value="${105*pi/180}"/> <!-- rad -->
+    <xacro:property name="hipFE_effort_limit" value="10927.0"/> <!-- IU -->
+    <xacro:property name="hipFE_velocity_limit" value="48.0"/> <!-- rad/s -->
+    <xacro:property name="hipAA_rotation_lower_limit" value="${20*pi/180}"/> <!-- rad -->
+    <xacro:property name="hipAA_rotation_upper_limit" value="${-30*pi/180}"/> <!-- rad -->
+    <xacro:property name="hipAA_effort_limit" value="10927.0"/> <!-- IU -->
+    <xacro:property name="hipAA_velocity_limit" value="15.0"/> <!-- rad/s -->
     <xacro:property name="knee_rotation_lower_limit" value="${-5*pi/180}"/>
     <xacro:property name="knee_rotation_upper_limit" value="${115*pi/180}"/>
@@ -43,13 +49,20 @@
     <joint name="hip" type="fixed">
         <parent link="${parent_name}"/>
-        <child link="hip_bone"/>
+        <child link="hip_base"/>
         <origin xyz="0 0 ${lower_leg_height+upper_leg_height+hover_height}" rpy="0 0 0"/>
     </joint>
-    <joint name="left_hip" type="revolute">
-        <parent link="hip_bone"/>
+    <joint name="left_hipAA" type="revolute">
+        <parent link="hip_base"/>
+        <child link="hip_moving_left"/>
+        <origin xyz="0 ${-hip_base_height/2} 0" rpy="0 0 0"/>
+        <axis xyz="1 0 0"/>
+        <limit velocity="${hipAA_velocity_limit}" effort="${hipAA_effort_limit}" lower="${hipAA_rotation_lower_limit}" upper="${hipAA_rotation_upper_limit}"/>
+    </joint>
+    <joint name="left_hipFE" type="revolute">
+        <parent link="hip_moving_left"/>
         <child link="upper_leg_left"/>
-        <origin xyz="0 ${-hip_height/2} 0" rpy="0 0 0"/>
+        <origin xyz="0 ${-hip_moving_height} 0" rpy="0 0 0"/>
         <axis xyz="0 1 0"/>
-        <limit velocity="${hip_velocity_limit}" effort="${hip_effort_limit}" lower="${hip_rotation_lower_limit}" upper="${hip_rotation_upper_limit}"/>
+        <limit velocity="${hipFE_velocity_limit}" effort="${hipFE_effort_limit}" lower="${hipFE_rotation_lower_limit}" upper="${hipFE_rotation_upper_limit}"/>
     </joint>
     <joint name="left_knee" type="revolute">
@@ -67,10 +80,17 @@
         <limit velocity="${ankle_velocity_limit}" effort="${ankle_effort_limit}" lower="${ankle_rotation_lower_limit}" upper="${ankle_rotation_upper_limit}"/>
     </joint>
-    <joint name="right_hip" type="revolute">
-        <parent link="hip_bone"/>
+    <joint name="right_hipAA" type="revolute">
+        <parent link="hip_base"/>
+        <child link="hip_moving_right"/>
+        <origin xyz="0 ${hip_base_height/2} 0" rpy="0 0 0"/>
+        <axis xyz="1 0 0"/>
+        <limit velocity="${hipAA_velocity_limit}" effort="${hipAA_effort_limit}" lower="${-hipAA_rotation_lower_limit}" upper="${-hipAA_rotation_upper_limit}"/>
+    </joint>
+    <joint name="right_hipFE" type="revolute">
+        <parent link="hip_moving_right"/>
         <child link="upper_leg_right"/>
-        <origin xyz="0 ${hip_height/2} 0" rpy="0 0 0"/>
+        <origin xyz="0 ${hip_moving_height} 0" rpy="0 0 0"/>
         <axis xyz="0 1 0"/>
-        <limit velocity="${hip_velocity_limit}" effort="${hip_effort_limit}" lower="${hip_rotation_lower_limit}" upper="${hip_rotation_upper_limit}"/>
+        <limit velocity="${hipFE_velocity_limit}" effort="${hipFE_effort_limit}" lower="${hipFE_rotation_lower_limit}" upper="${hipFE_rotation_upper_limit}"/>
     </joint>
     <joint name="right_knee" type="revolute">
@@ -89,5 +109,5 @@
     </joint>
     <!-- give colors to some links in gazebo -->
-    <gazebo reference="hip_bone">
+    <gazebo reference="hip_base">
         <material>Gazebo/Blue</material>
     </gazebo>
@@ -99,13 +119,30 @@
     </gazebo>
     <!-- Hip-->
-    <link name="hip_bone">
+    <link name="hip_base">
         <visual>
             <origin xyz="0 0 0" rpy="0 0 0"/>
             <geometry>
-                <box size="${width} ${hip_height} ${width}"/>
+                <box size="${width} ${hip_base_height} ${width}"/>
             </geometry>
         </visual>
         <inertial>
             <origin xyz="0 0 0" rpy="0 0 0"/>
+            <mass value="${mass}"/>
+            <inertia
+                    ixx="${mass / 12.0 * (width*width + lower_leg_height*lower_leg_height)}" ixy="0.0" ixz="0.0"
+                    iyy="${mass / 12.0 * (lower_leg_height*lower_leg_height + width*width)}" iyz="0.0"
+                    izz="${mass / 12.0 * (width*width + width*width)}"/>
+        </inertial>
+    </link>
+    <!-- Left Moving Hip-->
+    <link name="hip_moving_left">
+        <visual>
+            <origin xyz="0 ${-hip_moving_height/2} 0" rpy="0 0 0"/>
+            <geometry>
+                <box size="${width} ${hip_moving_height} ${width}"/>
+            </geometry>
+        </visual>
+        <inertial>
+            <origin xyz="0 ${hip_moving_height/2} 0" rpy="0 0 0"/>
             <mass value="${mass}"/>
             <inertia
@@ -137,5 +174,5 @@
     <link name="lower_leg_left">
         <visual>
-            <origin xyz="${-0.4*width} 0 ${-1.0*lower_leg_height}" rpy="0 0 1.8"/>
+            <origin xyz="0 0 ${-lower_leg_height/2}" rpy="0 0 1.8"/>
             <geometry>
                 <box size="${width} ${width} ${lower_leg_height}"/>
@@ -175,4 +212,21 @@
         </collision>
     </link>
+    <!-- Right Moving Hip-->
+    <link name="hip_moving_right">
+        <visual>
+            <origin xyz="0 ${hip_moving_height/2} 0" rpy="0 0 0"/>
+            <geometry>
+                <box size="${width} ${hip_moving_height} ${width}"/>
+            </geometry>
+        </visual>
+        <inertial>
+            <origin xyz="0 ${hip_moving_height/2} 0" rpy="0 0 0"/>
+            <mass value="${mass}"/>
+            <inertia
+                    ixx="${mass / 12.0 * (width*width + lower_leg_height*lower_leg_height)}" ixy="0.0" ixz="0.0"
+                    iyy="${mass / 12.0 * (lower_leg_height*lower_leg_height + width*width)}" iyz="0.0"
+                    izz="${mass / 12.0 * (width*width + width*width)}"/>
+        </inertial>
+    </link>
     <!-- Upper Leg Right-->
     <link name="upper_leg_right">

Commit message: Add new joint hip to transmission

File: march_ws/src/march_description/urdf/march-iii.xacro (robot description, xacro)
@@ -288,10 +288,20 @@
     </link>
     <!-- ROS Control plugin for Gazebo -->
-    <transmission name="left_hip">
-        <type>transmission_interface/SimpleTransmission</type>
-        <joint name="left_hip">
-            <hardwareInterface>hardware_interface/EffortJointInterface</hardwareInterface>
-        </joint>
-        <actuator name="left_hip_motor">
+    <transmission name="left_hipAA">
+        <type>transmission_interface/SimpleTransmission</type>
+        <joint name="left_hipAA">
+            <hardwareInterface>hardware_interface/EffortJointInterface</hardwareInterface>
+        </joint>
+        <actuator name="left_hipAA_motor">
+            <hardwareInterface>hardware_interface/EffortJointInterface</hardwareInterface>
+            <mechanicalReduction>1</mechanicalReduction>
+        </actuator>
+    </transmission>
+    <transmission name="left_hipFE">
+        <type>transmission_interface/SimpleTransmission</type>
+        <joint name="left_hipFE">
+            <hardwareInterface>hardware_interface/EffortJointInterface</hardwareInterface>
+        </joint>
+        <actuator name="left_hipFE_motor">
             <hardwareInterface>hardware_interface/EffortJointInterface</hardwareInterface>
             <mechanicalReduction>1</mechanicalReduction>
@@ -318,10 +328,20 @@
         </actuator>
     </transmission>
-    <transmission name="right_hip">
-        <type>transmission_interface/SimpleTransmission</type>
-        <joint name="right_hip">
-            <hardwareInterface>hardware_interface/EffortJointInterface</hardwareInterface>
-        </joint>
-        <actuator name="right_hip_motor">
+    <transmission name="right_hipAA">
+        <type>transmission_interface/SimpleTransmission</type>
+        <joint name="right_hipAA">
+            <hardwareInterface>hardware_interface/EffortJointInterface</hardwareInterface>
+        </joint>
+        <actuator name="right_hipAA_motor">
+            <hardwareInterface>hardware_interface/EffortJointInterface</hardwareInterface>
+            <mechanicalReduction>1</mechanicalReduction>
+        </actuator>
+    </transmission>
+    <transmission name="right_hipFE">
+        <type>transmission_interface/SimpleTransmission</type>
+        <joint name="right_hipFE">
+            <hardwareInterface>hardware_interface/EffortJointInterface</hardwareInterface>
+        </joint>
+        <actuator name="right_hipFE_motor">
             <hardwareInterface>hardware_interface/EffortJointInterface</hardwareInterface>
             <mechanicalReduction>1</mechanicalReduction>
