Commit message: Implement HAA joint with angle in base

File: march_ws/src/march_description/urdf/march-iii.xacro (robot description, xacro)
@@ -19,13 +19,14 @@
     <xacro:property name="hip_height" value="0.420"/>
     <xacro:property name="hip_base_height" value="0.160"/>
-    <xacro:property name="hip_moving_height" value="0.130"/>
-    <xacro:property name="hipFE_rotation_lower_limit" value="${-15*pi/180}"/> <!-- rad -->
-    <xacro:property name="hipFE_rotation_upper_limit" value="${105*pi/180}"/> <!-- rad -->
-    <xacro:property name="hipFE_effort_limit" value="10927.0"/> <!-- IU -->
-    <xacro:property name="hipFE_velocity_limit" value="48.0"/> <!-- rad/s -->
-    <xacro:property name="hipAA_rotation_lower_limit" value="${20*pi/180}"/> <!-- rad -->
-    <xacro:property name="hipAA_rotation_upper_limit" value="${-30*pi/180}"/> <!-- rad -->
-    <xacro:property name="hipAA_effort_limit" value="10927.0"/> <!-- IU -->
-    <xacro:property name="hipAA_velocity_limit" value="15.0"/> <!-- rad/s -->
+    <xacro:property name="hip_aa_frame_height" value="0.130"/>
+    <xacro:property name="hip_aa_frame_width" value="0.1395"/>
+    <xacro:property name="hip_fe_rotation_lower_limit" value="${-15*pi/180}"/> <!-- rad -->
+    <xacro:property name="hip_fe_rotation_upper_limit" value="${105*pi/180}"/> <!-- rad -->
+    <xacro:property name="hip_fe_effort_limit" value="10927.0"/> <!-- IU -->
+    <xacro:property name="hip_fe_velocity_limit" value="48.0"/> <!-- rad/s -->
+    <xacro:property name="hip_aa_rotation_lower_limit" value="${20*pi/180}"/> <!-- rad -->
+    <xacro:property name="hip_aa_rotation_upper_limit" value="${-30*pi/180}"/> <!-- rad -->
+    <xacro:property name="hip_aa_effort_limit" value="10927.0"/> <!-- IU -->
+    <xacro:property name="hip_aa_velocity_limit" value="15.0"/> <!-- rad/s -->
     <xacro:property name="knee_rotation_lower_limit" value="${-5*pi/180}"/>
     <xacro:property name="knee_rotation_upper_limit" value="${115*pi/180}"/>
@@ -46,5 +47,4 @@
     <!-- Used for fixing robot to Gazebo 'base_link' -->
     <link name="${parent_name}"/>
-<!--    TODO: Add the HAA joints!-->
     <joint name="hip" type="fixed">
         <parent link="${parent_name}"/>
@@ -52,17 +52,22 @@
         <origin xyz="0 0 ${lower_leg_height+upper_leg_height+hover_height}" rpy="0 0 0"/>
     </joint>
-    <joint name="left_hipAA" type="revolute">
+    <joint name="left_hip_aa" type="revolute">
         <parent link="hip_base"/>
-        <child link="hip_moving_left"/>
+        <child link="hip_aa_frame_left_side"/>
         <origin xyz="0 ${-hip_base_height/2} 0" rpy="0 0 0"/>
         <axis xyz="1 0 0"/>
-        <limit velocity="${hipAA_velocity_limit}" effort="${hipAA_effort_limit}" lower="${hipAA_rotation_lower_limit}" upper="${hipAA_rotation_upper_limit}"/>
-    </joint>
-    <joint name="left_hipFE" type="revolute">
-        <parent link="hip_moving_left"/>
+        <limit velocity="${hip_aa_velocity_limit}" effort="${hip_aa_effort_limit}" lower="${hip_aa_rotation_lower_limit}" upper="${hip_aa_rotation_upper_limit}"/>
+    </joint>
+    <joint name="left_hip_angle" type="fixed">
+        <parent link="hip_aa_frame_left_side"/>
+        <child link="hip_aa_frame_left_front"/>
+        <origin xyz="0 ${-hip_aa_frame_height} 0" rpy="0 0 0"/>
+    </joint>
+    <joint name="left_hip_fe" type="revolute">
+        <parent link="hip_aa_frame_left_front"/>
         <child link="upper_leg_left"/>
-        <origin xyz="0 ${-hip_moving_height} 0" rpy="0 0 0"/>
+        <origin xyz="${-hip_aa_frame_width} 0 0" rpy="0 0 0"/>
         <axis xyz="0 1 0"/>
-        <limit velocity="${hipFE_velocity_limit}" effort="${hipFE_effort_limit}" lower="${hipFE_rotation_lower_limit}" upper="${hipFE_rotation_upper_limit}"/>
+        <limit velocity="${hip_fe_velocity_limit}" effort="${hip_fe_effort_limit}" lower="${hip_fe_rotation_lower_limit}" upper="${hip_fe_rotation_upper_limit}"/>
     </joint>
     <joint name="left_knee" type="revolute">
@@ -80,17 +85,22 @@
         <limit velocity="${ankle_velocity_limit}" effort="${ankle_effort_limit}" lower="${ankle_rotation_lower_limit}" upper="${ankle_rotation_upper_limit}"/>
     </joint>
-    <joint name="right_hipAA" type="revolute">
+    <joint name="right_hip_aa" type="revolute">
         <parent link="hip_base"/>
-        <child link="hip_moving_right"/>
+        <child link="hip_aa_frame_right_side"/>
         <origin xyz="0 ${hip_base_height/2} 0" rpy="0 0 0"/>
         <axis xyz="1 0 0"/>
-        <limit velocity="${hipAA_velocity_limit}" effort="${hipAA_effort_limit}" lower="${-hipAA_rotation_lower_limit}" upper="${-hipAA_rotation_upper_limit}"/>
-    </joint>
-    <joint name="right_hipFE" type="revolute">
-        <parent link="hip_moving_right"/>
+        <limit velocity="${hip_aa_velocity_limit}" effort="${hip_aa_effort_limit}" lower="${-hip_aa_rotation_lower_limit}" upper="${-hip_aa_rotation_upper_limit}"/>
+    </joint>
+    <joint name="right_hip_angle" type="fixed">
+        <parent link="hip_aa_frame_right_side"/>
+        <child link="hip_aa_frame_right_front"/>
+        <origin xyz="0 ${hip_aa_frame_height} 0" rpy="0 0 0"/>
+    </joint>
+    <joint name="right_hip_fe" type="revolute">
+        <parent link="hip_aa_frame_right_front"/>
         <child link="upper_leg_right"/>
-        <origin xyz="0 ${hip_moving_height} 0" rpy="0 0 0"/>
+        <origin xyz="${-hip_aa_frame_width} 0 0" rpy="0 0 0"/>
         <axis xyz="0 1 0"/>
-        <limit velocity="${hipFE_velocity_limit}" effort="${hipFE_effort_limit}" lower="${hipFE_rotation_lower_limit}" upper="${hipFE_rotation_upper_limit}"/>
+        <limit velocity="${hip_fe_velocity_limit}" effort="${hip_fe_effort_limit}" lower="${hip_fe_rotation_lower_limit}" upper="${hip_fe_rotation_upper_limit}"/>
     </joint>
     <joint name="right_knee" type="revolute">
@@ -119,4 +129,5 @@
     </gazebo>
     <!-- Hip-->
+<!--    TODO: add angle in hip moving part -->
     <link name="hip_base">
         <visual>
@@ -136,13 +147,29 @@
     </link>
     <!-- Left Moving Hip-->
-    <link name="hip_moving_left">
-        <visual>
-            <origin xyz="0 ${-hip_moving_height/2} 0" rpy="0 0 0"/>
-            <geometry>
-                <box size="${width} ${hip_moving_height} ${width}"/>
-            </geometry>
-        </visual>
-        <inertial>
-            <origin xyz="0 ${hip_moving_height/2} 0" rpy="0 0 0"/>
+    <link name="hip_aa_frame_left_side">
+        <visual>
+            <origin xyz="0 ${-hip_aa_frame_height/2} 0" rpy="0 0 0"/>
+            <geometry>
+                <box size="${width} ${hip_aa_frame_height} ${width}"/>
+            </geometry>
+        </visual>
+        <inertial>
+            <origin xyz="0 ${hip_aa_frame_height/2} 0" rpy="0 0 0"/>
+            <mass value="${mass}"/>
+            <inertia
+                    ixx="${mass / 12.0 * (width*width + lower_leg_height*lower_leg_height)}" ixy="0.0" ixz="0.0"
+                    iyy="${mass / 12.0 * (lower_leg_height*lower_leg_height + width*width)}" iyz="0.0"
+                    izz="${mass / 12.0 * (width*width + width*width)}"/>
+        </inertial>
+    </link>
+    <link name="hip_aa_frame_left_front">
+        <visual>
+            <origin xyz="${-hip_aa_frame_width/2} 0 0" rpy="0 0 0"/>
+            <geometry>
+                <box size="${hip_aa_frame_width} ${width} ${width}"/>
+            </geometry>
+        </visual>
+        <inertial>
+            <origin xyz="${-hip_aa_frame_width/2} 0 0" rpy="0 0 0"/>
             <mass value="${mass}"/>
             <inertia
@@ -162,4 +189,10 @@
             </geometry>
         </visual>
+        <collision>
+            <origin xyz="0 0 ${-upper_leg_height/2}" rpy="0 0 0"/>
+            <geometry>
+                <box size="${width} ${width} ${upper_leg_height}"/>
+            </geometry>
+        </collision>
         <inertial>
             <origin xyz="0 0 ${-upper_leg_height/2}" rpy="0 0 0"/>
@@ -174,5 +207,5 @@
     <link name="lower_leg_left">
         <visual>
-            <origin xyz="0 0 ${-lower_leg_height/2}" rpy="0 0 1.8"/>
+            <origin xyz="0 0 ${-lower_leg_height/2}" rpy="0 0 0"/>
             <geometry>
                 <box size="${width} ${width} ${lower_leg_height}"/>
@@ -213,13 +246,29 @@
     </link>
     <!-- Right Moving Hip-->
-    <link name="hip_moving_right">
-        <visual>
-            <origin xyz="0 ${hip_moving_height/2} 0" rpy="0 0 0"/>
-            <geometry>
-                <box size="${width} ${hip_moving_height} ${width}"/>
-            </geometry>
-        </visual>
-        <inertial>
-            <origin xyz="0 ${hip_moving_height/2} 0" rpy="0 0 0"/>
+    <link name="hip_aa_frame_right_side">
+        <visual>
+            <origin xyz="0 ${hip_aa_frame_height/2} 0" rpy="0 0 0"/>
+            <geometry>
+                <box size="${width} ${hip_aa_frame_height} ${width}"/>
+            </geometry>
+        </visual>
+        <inertial>
+            <origin xyz="0 ${hip_aa_frame_height/2} 0" rpy="0 0 0"/>
+            <mass value="${mass}"/>
+            <inertia
+                    ixx="${mass / 12.0 * (width*width + lower_leg_height*lower_leg_height)}" ixy="0.0" ixz="0.0"
+                    iyy="${mass / 12.0 * (lower_leg_height*lower_leg_height + width*width)}" iyz="0.0"
+                    izz="${mass / 12.0 * (width*width + width*width)}"/>
+        </inertial>
+    </link>
+    <link name="hip_aa_frame_right_front">
+        <visual>
+            <origin xyz="${-hip_aa_frame_width/2} 0 0" rpy="0 0 0"/>
+            <geometry>
+                <box size="${hip_aa_frame_width} ${width} ${width}"/>
+            </geometry>
+        </visual>
+        <inertial>
+            <origin xyz="${-hip_aa_frame_width/2} 0 0" rpy="0 0 0"/>
             <mass value="${mass}"/>
             <inertia
@@ -238,4 +287,10 @@
             </geometry>
         </visual>
+        <collision>
+            <origin xyz="0 0 ${-upper_leg_height/2}" rpy="0 0 0"/>
+            <geometry>
+                <box size="${width} ${width} ${upper_leg_height}"/>
+            </geometry>
+        </collision>
         <inertial>
             <origin xyz="0 0 ${-upper_leg_height/2}" rpy="0 0 0"/>
@@ -288,20 +343,20 @@
     </link>
     <!-- ROS Control plugin for Gazebo -->
-    <transmission name="left_hipAA">
-        <type>transmission_interface/SimpleTransmission</type>
-        <joint name="left_hipAA">
-            <hardwareInterface>hardware_interface/EffortJointInterface</hardwareInterface>
-        </joint>
-        <actuator name="left_hipAA_motor">
-            <hardwareInterface>hardware_interface/EffortJointInterface</hardwareInterface>
-            <mechanicalReduction>1</mechanicalReduction>
-        </actuator>
-    </transmission>
-    <transmission name="left_hipFE">
-        <type>transmission_interface/SimpleTransmission</type>
-        <joint name="left_hipFE">
-            <hardwareInterface>hardware_interface/EffortJointInterface</hardwareInterface>
-        </joint>
-        <actuator name="left_hipFE_motor">
+    <transmission name="left_hip_aa">
+        <type>transmission_interface/SimpleTransmission</type>
+        <joint name="left_hip_aa">
+            <hardwareInterface>hardware_interface/EffortJointInterface</hardwareInterface>
+        </joint>
+        <actuator name="left_hip_aa_motor">
+            <hardwareInterface>hardware_interface/EffortJointInterface</hardwareInterface>
+            <mechanicalReduction>1</mechanicalReduction>
+        </actuator>
+    </transmission>
+    <transmission name="left_hip_fe">
+        <type>transmission_interface/SimpleTransmission</type>
+        <joint name="left_hip_fe">
+            <hardwareInterface>hardware_interface/EffortJointInterface</hardwareInterface>
+        </joint>
+        <actuator name="left_hip_fe_motor">
             <hardwareInterface>hardware_interface/EffortJointInterface</hardwareInterface>
             <mechanicalReduction>1</mechanicalReduction>
@@ -328,20 +383,20 @@
         </actuator>
     </transmission>
-    <transmission name="right_hipAA">
-        <type>transmission_interface/SimpleTransmission</type>
-        <joint name="right_hipAA">
-            <hardwareInterface>hardware_interface/EffortJointInterface</hardwareInterface>
-        </joint>
-        <actuator name="right_hipAA_motor">
-            <hardwareInterface>hardware_interface/EffortJointInterface</hardwareInterface>
-            <mechanicalReduction>1</mechanicalReduction>
-        </actuator>
-    </transmission>
-    <transmission name="right_hipFE">
-        <type>transmission_interface/SimpleTransmission</type>
-        <joint name="right_hipFE">
-            <hardwareInterface>hardware_interface/EffortJointInterface</hardwareInterface>
-        </joint>
-        <actuator name="right_hipFE_motor">
+    <transmission name="right_hip_aa">
+        <type>transmission_interface/SimpleTransmission</type>
+        <joint name="right_hip_aa">
+            <hardwareInterface>hardware_interface/EffortJointInterface</hardwareInterface>
+        </joint>
+        <actuator name="right_hip_aa_motor">
+            <hardwareInterface>hardware_interface/EffortJointInterface</hardwareInterface>
+            <mechanicalReduction>1</mechanicalReduction>
+        </actuator>
+    </transmission>
+    <transmission name="right_hip_fe">
+        <type>transmission_interface/SimpleTransmission</type>
+        <joint name="right_hip_fe">
+            <hardwareInterface>hardware_interface/EffortJointInterface</hardwareInterface>
+        </joint>
+        <actuator name="right_hip_fe_motor">
             <hardwareInterface>hardware_interface/EffortJointInterface</hardwareInterface>
             <mechanicalReduction>1</mechanicalReduction>

Commit message: Implement a distance between the ankle and the foot

File: march_ws/src/march_description/urdf/march-iii.xacro (robot description, xacro)
@@ -17,4 +17,5 @@
     <xacro:property name="foot_height" value="${0.184}"/>
     <xacro:property name="foot_mass" value="0.393"/>
+    <xacro:property name="ankle_plate_height" value="0.07"/>
     <xacro:property name="hip_height" value="0.420"/>
     <xacro:property name="hip_base_height" value="0.160"/>
@@ -80,8 +81,13 @@
     <joint name="left_ankle" type="revolute">
         <parent link="lower_leg_left"/>
-        <child link="foot_left"/>
+        <child link="ankle_plate_left"/>
         <origin xyz="0 0 ${-lower_leg_height}" rpy="0 0 0"/>
         <axis xyz="0 1 0"/>
         <limit velocity="${ankle_velocity_limit}" effort="${ankle_effort_limit}" lower="${ankle_rotation_lower_limit}" upper="${ankle_rotation_upper_limit}"/>
+    </joint>
+    <joint name="left_foot_angle" type="fixed">
+        <parent link="ankle_plate_left"/>
+        <child link="foot_left"/>
+        <origin xyz="0 0 ${-ankle_plate_height}" rpy="0 0 0"/>
     </joint>
     <joint name="right_hip_aa" type="revolute">
@@ -113,8 +119,13 @@
     <joint name="right_ankle" type="revolute">
         <parent link="lower_leg_right"/>
-        <child link="foot_right"/>
+        <child link="ankle_plate_right"/>
         <origin xyz="0 0 ${-lower_leg_height}" rpy="0 0 0"/>
         <axis xyz="0 1 0"/>
         <limit velocity="${ankle_velocity_limit}" effort="${ankle_effort_limit}" lower="${ankle_rotation_lower_limit}" upper="${ankle_rotation_upper_limit}"/>
+    </joint>
+    <joint name="right_foot_angle" type="fixed">
+        <parent link="ankle_plate_right"/>
+        <child link="foot_right"/>
+        <origin xyz="0 0 ${-ankle_plate_height}" rpy="0 0 0"/>
     </joint>
     <!-- give colors to some links in gazebo -->
@@ -222,4 +233,22 @@
         </inertial>
     </link>
+    <!-- Lower Leg Left -->
+    <link name="ankle_plate_left">
+        <visual>
+            <origin xyz="0 0 ${-ankle_plate_height/2}" rpy="0 0 0"/>
+            <geometry>
+                <box size="${width} ${width} ${ankle_plate_height}"/>
+                <!--                <mesh filename="package://march_description/urdf/stl-files/LowerLeg.stl" scale="1.2 1.2 1.2"/>-->
+            </geometry>
+        </visual>
+        <inertial>
+            <origin xyz="0 0 ${-ankle_plate_height/2}" rpy="0 0 0"/>
+            <mass value="${mass}"/>
+            <inertia
+                    ixx="${mass / 12.0 * (width*width + lower_leg_height*lower_leg_height)}" ixy="0.0" ixz="0.0"
+                    iyy="${mass / 12.0 * (lower_leg_height*lower_leg_height + width*width)}" iyz="0.0"
+                    izz="${mass / 12.0 * (width*width + width*width)}"/>
+        </inertial>
+    </link>
     <!-- Foot Left -->
     <link name="foot_left">
@@ -241,5 +270,4 @@
             <geometry>
                 <box size="${foot_height} ${width} ${width}"/>
-                <!--    TODO: The joint turns around this point, but the actual foot begins a little bit lower (70 mm?).-->
             </geometry>
         </collision>
@@ -319,4 +347,22 @@
         </inertial>
     </link>
+    <!-- Lower Leg Right -->
+    <link name="ankle_plate_right">
+        <visual>
+            <origin xyz="0 0 ${-ankle_plate_height/2}" rpy="0 0 0"/>
+            <geometry>
+                <box size="${width} ${width} ${ankle_plate_height}"/>
+                <!--                <mesh filename="package://march_description/urdf/stl-files/LowerLeg.stl" scale="1.2 1.2 1.2"/>-->
+            </geometry>
+        </visual>
+        <inertial>
+            <origin xyz="0 0 ${-ankle_plate_height/2}" rpy="0 0 0"/>
+            <mass value="${mass}"/>
+            <inertia
+                    ixx="${mass / 12.0 * (width*width + lower_leg_height*lower_leg_height)}" ixy="0.0" ixz="0.0"
+                    iyy="${mass / 12.0 * (lower_leg_height*lower_leg_height + width*width)}" iyz="0.0"
+                    izz="${mass / 12.0 * (width*width + width*width)}"/>
+        </inertial>
+    </link>
     <!-- Foot Right -->
     <link name="foot_right">
@@ -338,5 +384,4 @@
             <geometry>
                 <box size="${foot_height} ${width} ${width}"/>
-                <!--    TODO: The joint turns around this point, but the actual foot begins a little bit lower (70 mm?).-->
             </geometry>
         </collision>

Commit message: Add todo

File: march_ws/src/march_description/urdf/march-iii.xacro (robot description, xacro)
@@ -127,5 +127,5 @@
         <parent link="ankle_plate_right"/>
         <child link="foot_right"/>
-        <origin xyz="0 0 ${-ankle_plate_height}" rpy="0 0 0"/>
+        <origin xyz="0 0 ${-ankle_pslate_height}" rpy="0 0 0"/>
     </joint>
     <!-- give colors to some links in gazebo -->
@@ -140,5 +140,4 @@
     </gazebo>
     <!-- Hip-->
-<!--    TODO: add angle in hip moving part -->
     <link name="hip_base">
         <visual>
@@ -261,4 +260,5 @@
         <inertial>
             <origin xyz="${-foot_height/2} 0 0" rpy="0 0 0"/>
+<!--            TODO: adjust the origin so the foot also sticks out a little bit to the back-->
             <mass value="${foot_mass}"/>
             <inertia
@@ -375,4 +375,5 @@
         <inertial>
             <origin xyz="${-foot_height/2} 0 0" rpy="0 0 0"/>
+            <!--            TODO: adjust the origin so the foot also sticks out a little bit to the back-->
             <mass value="${mass}"/>
             <inertia
