Commit message: velocity limits increased, but lowered for the ankle

File: march_description/urdf/march-iv.xacro (robot description, xacro)
@@ -27,5 +27,5 @@
     <xacro:property name="hip_fe_soft_buffer" value="${3*pi/180}"/> <!-- rad -->
     <xacro:property name="hip_fe_effort_limit" value="10927.0"/> <!-- IU -->
-    <xacro:property name="hip_fe_velocity_limit" value="1.7"/> <!-- rad/s -->
+    <xacro:property name="hip_fe_velocity_limit" value="2.5"/> <!-- rad/s -->
     <xacro:property name="hip_aa_rotation_lower_limit" value="${-18*pi/180}"/> <!-- rad -->
     <xacro:property name="hip_aa_rotation_upper_limit" value="${17*pi/180}"/> <!-- rad -->
@@ -38,5 +38,5 @@
     <xacro:property name="knee_flexion_soft_buffer" value="${3*pi/180}"/> <!-- rad -->
     <xacro:property name="knee_effort_limit" value="10927.0"/>
-    <xacro:property name="knee_velocity_limit" value="1.7"/>
+    <xacro:property name="knee_velocity_limit" value="2.5"/>
     <xacro:property name="ankle_rotation_lower_limit" value="${-25*pi/180}"/>
     <xacro:property name="ankle_rotation_upper_limit" value="${15*pi/180}"/>
@@ -44,5 +44,5 @@
     <xacro:property name="ankle_plantarflexion_soft_buffer" value="${3*pi/180}"/> <!-- rad -->
     <xacro:property name="ankle_effort_limit" value="10927.0"/>
-    <xacro:property name="ankle_velocity_limit" value="1.0"/>
+    <xacro:property name="ankle_velocity_limit" value="0.6"/>
     <xacro:property name="hover_height" value="0.3"/>
     <xacro:property name="camera_link" value="0.05"/> <!-- Size of square 'camera' box -->

Commit message: change effort limits in xacro to higher value

File: march_description/urdf/march-iv.xacro (robot description, xacro)
@@ -26,10 +26,10 @@
     <xacro:property name="hip_fe_rotation_upper_limit" value="${100*pi/180}"/> <!-- rad -->
     <xacro:property name="hip_fe_soft_buffer" value="${3*pi/180}"/> <!-- rad -->
-    <xacro:property name="hip_fe_effort_limit" value="10927.0"/> <!-- IU -->
+    <xacro:property name="hip_fe_effort_limit" value="21840"/> <!-- IU -->
     <xacro:property name="hip_fe_velocity_limit" value="1.7"/> <!-- rad/s -->
     <xacro:property name="hip_aa_rotation_lower_limit" value="${-18*pi/180}"/> <!-- rad -->
     <xacro:property name="hip_aa_rotation_upper_limit" value="${17*pi/180}"/> <!-- rad -->
     <xacro:property name="hip_aa_soft_buffer" value="${5*pi/180}"/> <!-- rad -->
-    <xacro:property name="hip_aa_effort_limit" value="10927.0"/> <!-- IU -->
+    <xacro:property name="hip_aa_effort_limit" value="21840"/> <!-- IU -->
     <xacro:property name="hip_aa_velocity_limit" value="1.0"/> <!-- rad/s -->
     <xacro:property name="knee_rotation_lower_limit" value="${-5*pi/180}"/>
@@ -37,5 +37,5 @@
     <xacro:property name="knee_extension_soft_buffer" value="${4.5*pi/180}"/> <!-- rad -->
     <xacro:property name="knee_flexion_soft_buffer" value="${3*pi/180}"/> <!-- rad -->
-    <xacro:property name="knee_effort_limit" value="10927.0"/>
+    <xacro:property name="knee_effort_limit" value="21840"/>
     <xacro:property name="knee_velocity_limit" value="1.7"/>
     <xacro:property name="ankle_rotation_lower_limit" value="${-25*pi/180}"/>
@@ -43,5 +43,5 @@
     <xacro:property name="ankle_dorsalflexion_soft_buffer" value="${5*pi/180}"/> <!-- rad -->
     <xacro:property name="ankle_plantarflexion_soft_buffer" value="${3*pi/180}"/> <!-- rad -->
-    <xacro:property name="ankle_effort_limit" value="10927.0"/>
+    <xacro:property name="ankle_effort_limit" value="21840"/>
     <xacro:property name="ankle_velocity_limit" value="1.0"/>
     <xacro:property name="hover_height" value="0.3"/>
@@ -63,5 +63,5 @@
         <origin xyz="0 0 ${lower_leg_height+upper_leg_height+hover_height}" rpy="0 0 0"/>
     </joint>
-    <joint name="left_hip_aa" type="revolute">
+    <joint name="left_hip_aa" type="fixed">
         <parent link="hip_base"/>
         <child link="hip_aa_frame_left_side"/>
@@ -70,5 +70,5 @@
 <!-- TODO: @JitskedeVries  Improve k values-->
         <limit velocity="${hip_aa_velocity_limit}" effort="${hip_aa_effort_limit}" lower="${hip_aa_rotation_lower_limit}" upper="${hip_aa_rotation_upper_limit}"/>
-        <safety_controller soft_lower_limit="${hip_aa_rotation_lower_limit + hip_aa_soft_buffer}" soft_upper_limit="${hip_aa_rotation_upper_limit - hip_aa_soft_buffer}" k_position="5" k_velocity="5" />
+        <safety_controller soft_lower_limit="${hip_aa_rotation_lower_limit + hip_aa_soft_buffer}" soft_upper_limit="${hip_aa_rotation_upper_limit - hip_aa_soft_buffer}" k_position="5" k_velocity="20000" />
     </joint>
     <joint name="left_hip_angle" type="fixed">
@@ -83,5 +83,5 @@
         <axis xyz="0 1 0"/>
         <limit velocity="${hip_fe_velocity_limit}" effort="${hip_fe_effort_limit}" lower="${hip_fe_rotation_lower_limit}" upper="${hip_fe_rotation_upper_limit}"/>
-        <safety_controller soft_lower_limit="${hip_fe_rotation_lower_limit + hip_fe_soft_buffer}" soft_upper_limit="${hip_fe_rotation_upper_limit - hip_fe_soft_buffer}" k_position="5" k_velocity="5" />
+        <safety_controller soft_lower_limit="${hip_fe_rotation_lower_limit + hip_fe_soft_buffer}" soft_upper_limit="${hip_fe_rotation_upper_limit - hip_fe_soft_buffer}" k_position="5" k_velocity="20000" />
     </joint>
     <joint name="left_knee" type="revolute">
@@ -91,7 +91,7 @@
         <axis xyz="0 -1 0"/>
         <limit velocity="${knee_velocity_limit}" effort="${knee_effort_limit}" lower="${knee_rotation_lower_limit}" upper="${knee_rotation_upper_limit}"/>
-        <safety_controller soft_lower_limit="${knee_rotation_lower_limit + knee_extension_soft_buffer}" soft_upper_limit="${knee_rotation_upper_limit - knee_flexion_soft_buffer}" k_position="5" k_velocity="5" />
-    </joint>
-    <joint name="left_ankle" type="revolute">
+        <safety_controller soft_lower_limit="${knee_rotation_lower_limit + knee_extension_soft_buffer}" soft_upper_limit="${knee_rotation_upper_limit - knee_flexion_soft_buffer}" k_position="5" k_velocity="20000" />
+    </joint>
+    <joint name="left_ankle" type="fixed">
         <parent link="lower_leg_left"/>
         <child link="ankle_plate_left"/>
@@ -99,5 +99,5 @@
         <axis xyz="0 1 0"/>
         <limit velocity="${ankle_velocity_limit}" effort="${ankle_effort_limit}" lower="${ankle_rotation_lower_limit}" upper="${ankle_rotation_upper_limit}"/>
-        <safety_controller soft_lower_limit="${ankle_rotation_lower_limit + ankle_plantarflexion_soft_buffer}" soft_upper_limit="${ankle_rotation_upper_limit - ankle_dorsalflexion_soft_buffer}" k_position="5" k_velocity="5" />
+        <safety_controller soft_lower_limit="${ankle_rotation_lower_limit + ankle_plantarflexion_soft_buffer}" soft_upper_limit="${ankle_rotation_upper_limit - ankle_dorsalflexion_soft_buffer}" k_position="5" k_velocity="20000" />
     </joint>
     <joint name="left_foot_angle" type="fixed">
@@ -106,5 +106,5 @@
         <origin xyz="0 0 ${-ankle_plate_height}" rpy="0 0 0"/>
     </joint>
-    <joint name="right_hip_aa" type="revolute">
+    <joint name="right_hip_aa" type="fixed">
         <parent link="hip_base"/>
         <child link="hip_aa_frame_right_side"/>
@@ -112,5 +112,5 @@
         <axis xyz="1 0 0"/>
         <limit velocity="${hip_aa_velocity_limit}" effort="${hip_aa_effort_limit}" lower="${hip_aa_rotation_lower_limit}" upper="${hip_aa_rotation_upper_limit}"/>
-        <safety_controller soft_lower_limit="${hip_aa_rotation_lower_limit + hip_aa_soft_buffer}" soft_upper_limit="${hip_aa_rotation_upper_limit - hip_aa_soft_buffer}" k_position="5" k_velocity="5" />
+        <safety_controller soft_lower_limit="${hip_aa_rotation_lower_limit + hip_aa_soft_buffer}" soft_upper_limit="${hip_aa_rotation_upper_limit - hip_aa_soft_buffer}" k_position="5" k_velocity="20000" />
     </joint>
     <joint name="right_hip_angle" type="fixed">
@@ -125,5 +125,5 @@
         <axis xyz="0 1 0"/>
         <limit velocity="${hip_fe_velocity_limit}" effort="${hip_fe_effort_limit}" lower="${hip_fe_rotation_lower_limit}" upper="${hip_fe_rotation_upper_limit}"/>
-        <safety_controller soft_lower_limit="${hip_fe_rotation_lower_limit + hip_fe_soft_buffer}" soft_upper_limit="${hip_fe_rotation_upper_limit - hip_fe_soft_buffer}" k_position="5" k_velocity="5" />
+        <safety_controller soft_lower_limit="${hip_fe_rotation_lower_limit + hip_fe_soft_buffer}" soft_upper_limit="${hip_fe_rotation_upper_limit - hip_fe_soft_buffer}" k_position="5" k_velocity="20000" />
     </joint>
     <joint name="right_knee" type="revolute">
@@ -133,7 +133,7 @@
         <axis xyz="0 -1 0"/>
         <limit velocity="${knee_velocity_limit}" effort="${knee_effort_limit}" lower="${knee_rotation_lower_limit}" upper="${knee_rotation_upper_limit}"/>
-        <safety_controller soft_lower_limit="${knee_rotation_lower_limit + knee_extension_soft_buffer}" soft_upper_limit="${knee_rotation_upper_limit - knee_flexion_soft_buffer}" k_position="5" k_velocity="5" />
-    </joint>
-    <joint name="right_ankle" type="revolute">
+        <safety_controller soft_lower_limit="${knee_rotation_lower_limit + knee_extension_soft_buffer}" soft_upper_limit="${knee_rotation_upper_limit - knee_flexion_soft_buffer}" k_position="5" k_velocity="20000" />
+    </joint>
+    <joint name="right_ankle" type="fixed">
         <parent link="lower_leg_right"/>
         <child link="ankle_plate_right"/>
@@ -141,5 +141,5 @@
         <axis xyz="0 1 0"/>
         <limit velocity="${ankle_velocity_limit}" effort="${ankle_effort_limit}" lower="${ankle_rotation_lower_limit}" upper="${ankle_rotation_upper_limit}"/>
-        <safety_controller soft_lower_limit="${ankle_rotation_lower_limit + ankle_plantarflexion_soft_buffer}" soft_upper_limit="${ankle_rotation_upper_limit - ankle_dorsalflexion_soft_buffer}" k_position="5" k_velocity="5" />
+        <safety_controller soft_lower_limit="${ankle_rotation_lower_limit + ankle_plantarflexion_soft_buffer}" soft_upper_limit="${ankle_rotation_upper_limit - ankle_dorsalflexion_soft_buffer}" k_position="5" k_velocity="20000" />
     </joint>
     <joint name="right_foot_angle" type="fixed">

Commit message: Revert "change effort limits in xacro to higher value"
This reverts commit a84b58a1

File: march_description/urdf/march-iv.xacro (robot description, xacro)
@@ -26,10 +26,10 @@
     <xacro:property name="hip_fe_rotation_upper_limit" value="${100*pi/180}"/> <!-- rad -->
     <xacro:property name="hip_fe_soft_buffer" value="${3*pi/180}"/> <!-- rad -->
-    <xacro:property name="hip_fe_effort_limit" value="21840"/> <!-- IU -->
+    <xacro:property name="hip_fe_effort_limit" value="10927.0"/> <!-- IU -->
     <xacro:property name="hip_fe_velocity_limit" value="1.7"/> <!-- rad/s -->
     <xacro:property name="hip_aa_rotation_lower_limit" value="${-18*pi/180}"/> <!-- rad -->
     <xacro:property name="hip_aa_rotation_upper_limit" value="${17*pi/180}"/> <!-- rad -->
     <xacro:property name="hip_aa_soft_buffer" value="${5*pi/180}"/> <!-- rad -->
-    <xacro:property name="hip_aa_effort_limit" value="21840"/> <!-- IU -->
+    <xacro:property name="hip_aa_effort_limit" value="10927.0"/> <!-- IU -->
     <xacro:property name="hip_aa_velocity_limit" value="1.0"/> <!-- rad/s -->
     <xacro:property name="knee_rotation_lower_limit" value="${-5*pi/180}"/>
@@ -37,5 +37,5 @@
     <xacro:property name="knee_extension_soft_buffer" value="${4.5*pi/180}"/> <!-- rad -->
     <xacro:property name="knee_flexion_soft_buffer" value="${3*pi/180}"/> <!-- rad -->
-    <xacro:property name="knee_effort_limit" value="21840"/>
+    <xacro:property name="knee_effort_limit" value="10927.0"/>
     <xacro:property name="knee_velocity_limit" value="1.7"/>
     <xacro:property name="ankle_rotation_lower_limit" value="${-25*pi/180}"/>
@@ -43,5 +43,5 @@
     <xacro:property name="ankle_dorsalflexion_soft_buffer" value="${5*pi/180}"/> <!-- rad -->
     <xacro:property name="ankle_plantarflexion_soft_buffer" value="${3*pi/180}"/> <!-- rad -->
-    <xacro:property name="ankle_effort_limit" value="21840"/>
+    <xacro:property name="ankle_effort_limit" value="10927.0"/>
     <xacro:property name="ankle_velocity_limit" value="1.0"/>
     <xacro:property name="hover_height" value="0.3"/>
@@ -63,5 +63,5 @@
         <origin xyz="0 0 ${lower_leg_height+upper_leg_height+hover_height}" rpy="0 0 0"/>
     </joint>
-    <joint name="left_hip_aa" type="fixed">
+    <joint name="left_hip_aa" type="revolute">
         <parent link="hip_base"/>
         <child link="hip_aa_frame_left_side"/>
@@ -70,5 +70,5 @@
 <!-- TODO: @JitskedeVries  Improve k values-->
         <limit velocity="${hip_aa_velocity_limit}" effort="${hip_aa_effort_limit}" lower="${hip_aa_rotation_lower_limit}" upper="${hip_aa_rotation_upper_limit}"/>
-        <safety_controller soft_lower_limit="${hip_aa_rotation_lower_limit + hip_aa_soft_buffer}" soft_upper_limit="${hip_aa_rotation_upper_limit - hip_aa_soft_buffer}" k_position="5" k_velocity="20000" />
+        <safety_controller soft_lower_limit="${hip_aa_rotation_lower_limit + hip_aa_soft_buffer}" soft_upper_limit="${hip_aa_rotation_upper_limit - hip_aa_soft_buffer}" k_position="5" k_velocity="5" />
     </joint>
     <joint name="left_hip_angle" type="fixed">
@@ -83,5 +83,5 @@
         <axis xyz="0 1 0"/>
         <limit velocity="${hip_fe_velocity_limit}" effort="${hip_fe_effort_limit}" lower="${hip_fe_rotation_lower_limit}" upper="${hip_fe_rotation_upper_limit}"/>
-        <safety_controller soft_lower_limit="${hip_fe_rotation_lower_limit + hip_fe_soft_buffer}" soft_upper_limit="${hip_fe_rotation_upper_limit - hip_fe_soft_buffer}" k_position="5" k_velocity="20000" />
+        <safety_controller soft_lower_limit="${hip_fe_rotation_lower_limit + hip_fe_soft_buffer}" soft_upper_limit="${hip_fe_rotation_upper_limit - hip_fe_soft_buffer}" k_position="5" k_velocity="5" />
     </joint>
     <joint name="left_knee" type="revolute">
@@ -91,7 +91,7 @@
         <axis xyz="0 -1 0"/>
         <limit velocity="${knee_velocity_limit}" effort="${knee_effort_limit}" lower="${knee_rotation_lower_limit}" upper="${knee_rotation_upper_limit}"/>
-        <safety_controller soft_lower_limit="${knee_rotation_lower_limit + knee_extension_soft_buffer}" soft_upper_limit="${knee_rotation_upper_limit - knee_flexion_soft_buffer}" k_position="5" k_velocity="20000" />
-    </joint>
-    <joint name="left_ankle" type="fixed">
+        <safety_controller soft_lower_limit="${knee_rotation_lower_limit + knee_extension_soft_buffer}" soft_upper_limit="${knee_rotation_upper_limit - knee_flexion_soft_buffer}" k_position="5" k_velocity="5" />
+    </joint>
+    <joint name="left_ankle" type="revolute">
         <parent link="lower_leg_left"/>
         <child link="ankle_plate_left"/>
@@ -99,5 +99,5 @@
         <axis xyz="0 1 0"/>
         <limit velocity="${ankle_velocity_limit}" effort="${ankle_effort_limit}" lower="${ankle_rotation_lower_limit}" upper="${ankle_rotation_upper_limit}"/>
-        <safety_controller soft_lower_limit="${ankle_rotation_lower_limit + ankle_plantarflexion_soft_buffer}" soft_upper_limit="${ankle_rotation_upper_limit - ankle_dorsalflexion_soft_buffer}" k_position="5" k_velocity="20000" />
+        <safety_controller soft_lower_limit="${ankle_rotation_lower_limit + ankle_plantarflexion_soft_buffer}" soft_upper_limit="${ankle_rotation_upper_limit - ankle_dorsalflexion_soft_buffer}" k_position="5" k_velocity="5" />
     </joint>
     <joint name="left_foot_angle" type="fixed">
@@ -106,5 +106,5 @@
         <origin xyz="0 0 ${-ankle_plate_height}" rpy="0 0 0"/>
     </joint>
-    <joint name="right_hip_aa" type="fixed">
+    <joint name="right_hip_aa" type="revolute">
         <parent link="hip_base"/>
         <child link="hip_aa_frame_right_side"/>
@@ -112,5 +112,5 @@
         <axis xyz="1 0 0"/>
         <limit velocity="${hip_aa_velocity_limit}" effort="${hip_aa_effort_limit}" lower="${hip_aa_rotation_lower_limit}" upper="${hip_aa_rotation_upper_limit}"/>
-        <safety_controller soft_lower_limit="${hip_aa_rotation_lower_limit + hip_aa_soft_buffer}" soft_upper_limit="${hip_aa_rotation_upper_limit - hip_aa_soft_buffer}" k_position="5" k_velocity="20000" />
+        <safety_controller soft_lower_limit="${hip_aa_rotation_lower_limit + hip_aa_soft_buffer}" soft_upper_limit="${hip_aa_rotation_upper_limit - hip_aa_soft_buffer}" k_position="5" k_velocity="5" />
     </joint>
     <joint name="right_hip_angle" type="fixed">
@@ -125,5 +125,5 @@
         <axis xyz="0 1 0"/>
         <limit velocity="${hip_fe_velocity_limit}" effort="${hip_fe_effort_limit}" lower="${hip_fe_rotation_lower_limit}" upper="${hip_fe_rotation_upper_limit}"/>
-        <safety_controller soft_lower_limit="${hip_fe_rotation_lower_limit + hip_fe_soft_buffer}" soft_upper_limit="${hip_fe_rotation_upper_limit - hip_fe_soft_buffer}" k_position="5" k_velocity="20000" />
+        <safety_controller soft_lower_limit="${hip_fe_rotation_lower_limit + hip_fe_soft_buffer}" soft_upper_limit="${hip_fe_rotation_upper_limit - hip_fe_soft_buffer}" k_position="5" k_velocity="5" />
     </joint>
     <joint name="right_knee" type="revolute">
@@ -133,7 +133,7 @@
         <axis xyz="0 -1 0"/>
         <limit velocity="${knee_velocity_limit}" effort="${knee_effort_limit}" lower="${knee_rotation_lower_limit}" upper="${knee_rotation_upper_limit}"/>
-        <safety_controller soft_lower_limit="${knee_rotation_lower_limit + knee_extension_soft_buffer}" soft_upper_limit="${knee_rotation_upper_limit - knee_flexion_soft_buffer}" k_position="5" k_velocity="20000" />
-    </joint>
-    <joint name="right_ankle" type="fixed">
+        <safety_controller soft_lower_limit="${knee_rotation_lower_limit + knee_extension_soft_buffer}" soft_upper_limit="${knee_rotation_upper_limit - knee_flexion_soft_buffer}" k_position="5" k_velocity="5" />
+    </joint>
+    <joint name="right_ankle" type="revolute">
         <parent link="lower_leg_right"/>
         <child link="ankle_plate_right"/>
@@ -141,5 +141,5 @@
         <axis xyz="0 1 0"/>
         <limit velocity="${ankle_velocity_limit}" effort="${ankle_effort_limit}" lower="${ankle_rotation_lower_limit}" upper="${ankle_rotation_upper_limit}"/>
-        <safety_controller soft_lower_limit="${ankle_rotation_lower_limit + ankle_plantarflexion_soft_buffer}" soft_upper_limit="${ankle_rotation_upper_limit - ankle_dorsalflexion_soft_buffer}" k_position="5" k_velocity="20000" />
+        <safety_controller soft_lower_limit="${ankle_rotation_lower_limit + ankle_plantarflexion_soft_buffer}" soft_upper_limit="${ankle_rotation_upper_limit - ankle_dorsalflexion_soft_buffer}" k_position="5" k_velocity="5" />
     </joint>
     <joint name="right_foot_angle" type="fixed">

Commit message: Don't launch left_hip_aa

File: march_description/urdf/march-iv.xacro (robot description, xacro)
@@ -63,5 +63,5 @@
         <origin xyz="0 0 ${lower_leg_height+upper_leg_height+hover_height}" rpy="0 0 0"/>
     </joint>
-    <joint name="left_hip_aa" type="revolute">
+    <joint name="left_hip_aa" type="fixed">
         <parent link="hip_base"/>
         <child link="hip_aa_frame_left_side"/>

Commit message: Update march_description/urdf/march-iv.xacro

File: march_description/urdf/march-iv.xacro (robot description, xacro)
@@ -63,5 +63,5 @@
         <origin xyz="0 0 ${lower_leg_height+upper_leg_height+hover_height}" rpy="0 0 0"/>
     </joint>
-    <joint name="left_hip_aa" type="fixed">
+    <joint name="left_hip_aa" type="revolute">
         <parent link="hip_base"/>
         <child link="hip_aa_frame_left_side"/>

Commit message: Change knee_extension_soft_buffer from 4.5 to 2
Worked during training

File: march_description/urdf/march-iv.xacro (robot description, xacro)
@@ -39,5 +39,5 @@
     <xacro:property name="knee_rotation_lower_limit" value="${-5*pi/180}"/>
     <xacro:property name="knee_rotation_upper_limit" value="${115*pi/180}"/>
-    <xacro:property name="knee_extension_soft_buffer" value="${4.5*pi/180}"/> <!-- rad -->
+    <xacro:property name="knee_extension_soft_buffer" value="${2*pi/180}"/> <!-- rad -->
     <xacro:property name="knee_flexion_soft_buffer" value="${3*pi/180}"/> <!-- rad -->
     <xacro:property name="knee_effort_limit" value="${max_effort_value}"/> <!-- IU = 20 A -->

Commit message: reduce haa buffer to 3.5

File: march_description/urdf/march-iv.xacro (robot description, xacro)
@@ -34,5 +34,5 @@
     <xacro:property name="hip_aa_rotation_lower_limit" value="${-18*pi/180}"/> <!-- rad -->
     <xacro:property name="hip_aa_rotation_upper_limit" value="${17*pi/180}"/> <!-- rad -->
-    <xacro:property name="hip_aa_soft_buffer" value="${5*pi/180}"/> <!-- rad -->
+    <xacro:property name="hip_aa_soft_buffer" value="${3.5*pi/180}"/> <!-- rad -->
     <xacro:property name="hip_aa_effort_limit" value="${max_effort_value}"/> <!-- IU = 20 A -->
     <xacro:property name="hip_aa_velocity_limit" value="1.0"/> <!-- rad/s -->

Commit message: Adjust walk_small to match new StoppableState structure.

File: march_description/urdf/march-iv.xacro (robot description, xacro)
@@ -12,14 +12,13 @@
     <xacro:property name="k_velocity_value" value="$(arg k_velocity_value)" />
     <!-- Constants for robot dimensions -->
-    <!-- TODO @Jitske: add accurate masses and inertia for all links -->
-    <xacro:property name="mass" value="1"/> <!-- arbitrary value for mass -->
+    <xacro:property name="mass" value="1"/>
     <xacro:property name="width" value="0.05"/> <!-- Square dimensions (widthxwidth) of beams -->
     <xacro:property name="upper_leg_height" value="${0.385}"/>
-    <xacro:property name="upper_leg_mass" value="1.080"/>
+    <xacro:property name="upper_leg_mass" value="6.860"/>
     <xacro:property name="lower_leg_height" value="${0.385}"/>
-    <xacro:property name="lower_leg_mass" value="1.133"/>
+    <xacro:property name="lower_leg_mass" value="2.637"/>
     <xacro:property name="foot_height_forward" value="${0.184}"/>
     <xacro:property name="foot_height_backward" value="${0.059}"/>
-    <xacro:property name="foot_mass" value="0.393"/>
+    <xacro:property name="foot_mass" value="0.847"/>
     <xacro:property name="ankle_plate_height" value="0.07"/>
     <xacro:property name="hip_height" value="0.420"/>
@@ -69,10 +68,7 @@
     <joint name="left_hip_aa" type="revolute">
         <parent link="hip_base"/>
-        <child link="hip_aa_frame_left_side"/>
+        <child link="hip_aa_//frame_left_side"/>
         <origin xyz="0 ${-hip_base_height/2} 0" rpy="0 0 0"/>
         <axis xyz="-1 0 0"/>
-<!-- TODO: @JitskedeVries  Improve k values-->
-        <limit velocity="${hip_aa_velocity_limit}" effort="${hip_aa_effort_limit}" lower="${hip_aa_rotation_lower_limit}" upper="${hip_aa_rotation_upper_limit}"/>
-        <safety_controller soft_lower_limit="${hip_aa_rotation_lower_limit + hip_aa_soft_buffer}" soft_upper_limit="${hip_aa_rotation_upper_limit - hip_aa_soft_buffer}" k_position="5" k_velocity="${k_velocity_value}" />
     </joint>
     <joint name="left_hip_angle" type="fixed">
@@ -274,5 +270,5 @@
         </collision>
     </link>
-    <!-- Lower Leg Left -->
+    <!-- Ankle plate Left -->
     <link name="ankle_plate_left">
         <visual>
