Commit message: Tune the max effort values for the simulation. This prevents safety controller from glitching, allowing replacement of endstops.

File: march_description/urdf/march-iv.xacro (robot description, xacro)
@@ -3,14 +3,22 @@
 <robot name="march" xmlns:xacro="http://www.ros.org/wiki/xacro">
     <!-- Switch between airgaiting or standing on the ground-->
-    <!--Value set to: 'world' fixes the robot to the world-->
-    <!--Value set to: 'base_link' makes the robot stand on the ground-->
-    <!--Important note: when changing value make sure rviz fixed frame is set to the same value (moveit.rviz)-->
+    <!-- Value set to: 'world' fixes the robot to the world-->
+    <!-- Value set to: 'base_link' makes the robot stand on the ground-->
+    <!-- Important note: when changing value make sure rviz fixed frame is set to the same value (moveit.rviz)-->
     <xacro:property name="parent_name" value="world"/>
+    <xacro:property name="hover_height" value="0.3"/>
     <xacro:arg name="max_effort_rotary" default="20475" /> <!-- = 25 A -->
     <xacro:arg name="max_effort_linear" default="22932.0" />  <!-- = 28 A -->
     <xacro:property name="max_effort_rotary" value="$(arg max_effort_rotary)" />
     <xacro:property name="max_effort_linear" value="$(arg max_effort_linear)" />
-    <xacro:arg name="k_velocity_value" default="20000.0" />
-    <xacro:property name="k_velocity_value" value="$(arg k_velocity_value)" />
+    <!-- Values for the safety limits, see https://wiki.ros.org/pr2_controller_manager/safety_limits -->
+    <xacro:arg name="k_velocity_value_rotary" default="20000.0" />
+    <xacro:arg name="k_velocity_value_linear" default="20000.0" />
+    <xacro:property name="k_velocity_value_rotary" value="$(arg k_velocity_value_rotary)" />
+    <xacro:property name="k_velocity_value_linear" value="$(arg k_velocity_value_linear)" />
+    <xacro:arg name="k_position_value_rotary" default="5.0" />
+    <xacro:arg name="k_position_value_linear" default="5.0" />
+    <xacro:property name="k_position_value_rotary" value="$(arg k_position_value_rotary)" />
+    <xacro:property name="k_position_value_linear" value="$(arg k_position_value_linear)" />
     <!-- Constants for robot dimensions -->
     <!-- Masses determined in https://confluence.projectmarch.nl:8443/display/41TECH/Weights+of+the+Exoskeleton -->
@@ -33,4 +41,8 @@
     <xacro:property name="foot_height_backward" value="${0.059}"/>
     <xacro:property name="foot_mass" value="0.847"/>
+    <xacro:property name="foot_mu1" value="0.9"/>
+    <xacro:property name="foot_mu2" value="0.9"/>
+    <!-- Minimum allowable depth before contact correction impulse is applied. -->
+    <xacro:property name="foot_min_depth" value="0.0005"/>
     <!-- mass = Passive ankle + foot -->
     <!-- Center of Mass (CoM) of the parts -->
@@ -115,5 +127,4 @@
     <xacro:property name="ankle_effort_limit" value="${max_effort_linear}"/> <!-- IU = 20 A -->
     <xacro:property name="ankle_velocity_limit" value="1.0"/>
-    <xacro:property name="hover_height" value="0.3"/>
     <xacro:property name="camera_link" value="0.05"/> <!-- Size of square 'camera' box -->
     <xacro:property name="axel_offset" value="0.05"/> <!-- Space btw top of beam and the each joint -->
@@ -123,7 +134,4 @@
         <color rgba="0 0 0.6 1"/>
     </material>
-    <plugin name="gazebo_ros_control" filename="libgazebo_ros_control.so">
-        <robotNamespace>/march</robotNamespace>
-    </plugin>
     <!-- Used for fixing robot to Gazebo 'base_link' -->
     <link name="${parent_name}"/>
@@ -281,4 +289,9 @@
         </collision>
     </link>
+    <gazebo reference="foot_left">
+        <mu1>${foot_mu1}</mu1>
+        <mu2>${foot_mu2}</mu2>
+        <minDepth>${foot_min_depth}</minDepth>
+    </gazebo>
     <!-- Right Moving Hip-->
     <link name="hip_aa_frame_right_side">
@@ -406,9 +419,14 @@
         </collision>
     </link>
+    <gazebo reference="foot_right">
+        <mu1>${foot_mu1}</mu1>
+        <mu2>${foot_mu2}</mu2>
+        <minDepth>${foot_min_depth}</minDepth>
+    </gazebo>
     <!-- Joints -->
     <joint name="hip" type="fixed">
         <parent link="${parent_name}"/>
         <child link="hip_base"/>
-        <origin xyz="0 0 ${lower_leg_height+upper_leg_height+hover_height}" rpy="0 0 0"/>
+        <origin xyz="0 0 ${lower_leg_height+upper_leg_height+ankle_plate_height+width/2.0+hover_height}" rpy="0 0 0"/>
     </joint>
     <joint name="left_hip_aa" type="revolute">
@@ -417,6 +435,12 @@
         <origin xyz="0 ${-hip_base_height/2} 0" rpy="0 0 0"/>
         <axis xyz="-1 0 0"/>
-        <limit velocity="${hip_aa_velocity_limit}" effort="${hip_aa_effort_limit}" lower="${hip_aa_rotation_lower_limit}" upper="${hip_aa_rotation_upper_limit}"/>
-        <safety_controller soft_lower_limit="${hip_aa_rotation_lower_limit + hip_aa_soft_buffer}" soft_upper_limit="${hip_aa_rotation_upper_limit - hip_aa_soft_buffer}" k_position="5" k_velocity="${k_velocity_value}" />
+        <limit velocity="${hip_aa_velocity_limit}"
+               effort="${hip_aa_effort_limit}"
+               lower="${hip_aa_rotation_lower_limit}"
+               upper="${hip_aa_rotation_upper_limit}"/>
+        <safety_controller soft_lower_limit="${hip_aa_rotation_lower_limit + hip_aa_soft_buffer}"
+                           soft_upper_limit="${hip_aa_rotation_upper_limit - hip_aa_soft_buffer}"
+                           k_position="${k_position_value_linear}"
+                           k_velocity="${k_velocity_value_linear}" />
     </joint>
     <joint name="left_hip_angle" type="fixed">
@@ -430,6 +454,12 @@
         <origin xyz="${-hip_aa_frame_width} 0 0" rpy="0 0 0"/>
         <axis xyz="0 1 0"/>
-        <limit velocity="${hip_fe_velocity_limit}" effort="${hip_fe_effort_limit}" lower="${hip_fe_rotation_lower_limit}" upper="${hip_fe_rotation_upper_limit}"/>
-        <safety_controller soft_lower_limit="${hip_fe_rotation_lower_limit + hip_fe_soft_buffer}" soft_upper_limit="${hip_fe_rotation_upper_limit - hip_fe_soft_buffer}" k_position="5" k_velocity="${k_velocity_value}" />
+        <limit velocity="${hip_fe_velocity_limit}"
+               effort="${hip_fe_effort_limit}"
+               lower="${hip_fe_rotation_lower_limit}"
+               upper="${hip_fe_rotation_upper_limit}"/>
+        <safety_controller soft_lower_limit="${hip_fe_rotation_lower_limit + hip_fe_soft_buffer}"
+                           soft_upper_limit="${hip_fe_rotation_upper_limit - hip_fe_soft_buffer}"
+                           k_position="${k_position_value_rotary}"
+                           k_velocity="${k_velocity_value_rotary}" />
     </joint>
     <joint name="left_knee" type="revolute">
@@ -438,6 +468,12 @@
         <origin xyz="0 0 ${-upper_leg_height}" rpy="0 0 0"/>
         <axis xyz="0 -1 0"/>
-        <limit velocity="${knee_velocity_limit}" effort="${knee_effort_limit}" lower="${knee_rotation_lower_limit}" upper="${knee_rotation_upper_limit}"/>
-        <safety_controller soft_lower_limit="${knee_rotation_lower_limit + knee_extension_soft_buffer}" soft_upper_limit="${knee_rotation_upper_limit - knee_flexion_soft_buffer}" k_position="5" k_velocity="${k_velocity_value}" />
+        <limit velocity="${knee_velocity_limit}"
+               effort="${knee_effort_limit}"
+               lower="${knee_rotation_lower_limit}"
+               upper="${knee_rotation_upper_limit}"/>
+        <safety_controller soft_lower_limit="${knee_rotation_lower_limit + knee_extension_soft_buffer}"
+                           soft_upper_limit="${knee_rotation_upper_limit - knee_flexion_soft_buffer}"
+                           k_position="${k_position_value_rotary}"
+                           k_velocity="${k_velocity_value_rotary}" />
     </joint>
     <joint name="left_ankle" type="revolute">
@@ -446,6 +482,12 @@
         <origin xyz="0 0 ${-lower_leg_height}" rpy="0 0 0"/>
         <axis xyz="0 1 0"/>
-        <limit velocity="${ankle_velocity_limit}" effort="${ankle_effort_limit}" lower="${ankle_rotation_lower_limit}" upper="${ankle_rotation_upper_limit}"/>
-        <safety_controller soft_lower_limit="${ankle_rotation_lower_limit + ankle_plantarflexion_soft_buffer}" soft_upper_limit="${ankle_rotation_upper_limit - ankle_dorsalflexion_soft_buffer}" k_position="5" k_velocity="${k_velocity_value}" />
+        <limit velocity="${ankle_velocity_limit}"
+               effort="${ankle_effort_limit}"
+               lower="${ankle_rotation_lower_limit}"
+               upper="${ankle_rotation_upper_limit}"/>
+        <safety_controller soft_lower_limit="${ankle_rotation_lower_limit + ankle_plantarflexion_soft_buffer}"
+                           soft_upper_limit="${ankle_rotation_upper_limit - ankle_dorsalflexion_soft_buffer}"
+                           k_position="${k_position_value_linear}"
+                           k_velocity="${k_velocity_value_linear}" />
     </joint>
     <joint name="left_foot_angle" type="fixed">
@@ -459,6 +501,12 @@
         <origin xyz="0 ${hip_base_height/2} 0" rpy="0 0 0"/>
         <axis xyz="1 0 0"/>
-        <limit velocity="${hip_aa_velocity_limit}" effort="${hip_aa_effort_limit}" lower="${hip_aa_rotation_lower_limit}" upper="${hip_aa_rotation_upper_limit}"/>
-        <safety_controller soft_lower_limit="${hip_aa_rotation_lower_limit + hip_aa_soft_buffer}" soft_upper_limit="${hip_aa_rotation_upper_limit - hip_aa_soft_buffer}" k_position="5" k_velocity="${k_velocity_value}" />
+        <limit velocity="${hip_aa_velocity_limit}"
+               effort="${hip_aa_effort_limit}"
+               lower="${hip_aa_rotation_lower_limit}"
+               upper="${hip_aa_rotation_upper_limit}"/>
+        <safety_controller soft_lower_limit="${hip_aa_rotation_lower_limit + hip_aa_soft_buffer}"
+                           soft_upper_limit="${hip_aa_rotation_upper_limit - hip_aa_soft_buffer}"
+                           k_position="${k_position_value_linear}"
+                           k_velocity="${k_velocity_value_linear}" />
     </joint>
     <joint name="right_hip_angle" type="fixed">
@@ -472,6 +520,12 @@
         <origin xyz="${-hip_aa_frame_width} 0 0" rpy="0 0 0"/>
         <axis xyz="0 1 0"/>
-        <limit velocity="${hip_fe_velocity_limit}" effort="${hip_fe_effort_limit}" lower="${hip_fe_rotation_lower_limit}" upper="${hip_fe_rotation_upper_limit}"/>
-        <safety_controller soft_lower_limit="${hip_fe_rotation_lower_limit + hip_fe_soft_buffer}" soft_upper_limit="${hip_fe_rotation_upper_limit - hip_fe_soft_buffer}" k_position="5" k_velocity="${k_velocity_value}" />
+        <limit velocity="${hip_fe_velocity_limit}"
+               effort="${hip_fe_effort_limit}"
+               lower="${hip_fe_rotation_lower_limit}"
+               upper="${hip_fe_rotation_upper_limit}"/>
+        <safety_controller soft_lower_limit="${hip_fe_rotation_lower_limit + hip_fe_soft_buffer}"
+                           soft_upper_limit="${hip_fe_rotation_upper_limit - hip_fe_soft_buffer}"
+                           k_position="${k_position_value_rotary}"
+                           k_velocity="${k_velocity_value_rotary}" />
     </joint>
     <joint name="right_knee" type="revolute">
@@ -480,6 +534,12 @@
         <origin xyz="0 0 ${-upper_leg_height}" rpy="0 0 0"/>
         <axis xyz="0 -1 0"/>
-        <limit velocity="${knee_velocity_limit}" effort="${knee_effort_limit}" lower="${knee_rotation_lower_limit}" upper="${knee_rotation_upper_limit}"/>
-        <safety_controller soft_lower_limit="${knee_rotation_lower_limit + knee_extension_soft_buffer}" soft_upper_limit="${knee_rotation_upper_limit - knee_flexion_soft_buffer}" k_position="5" k_velocity="${k_velocity_value}" />
+        <limit velocity="${knee_velocity_limit}"
+               effort="${knee_effort_limit}"
+               lower="${knee_rotation_lower_limit}"
+               upper="${knee_rotation_upper_limit}"/>
+        <safety_controller soft_lower_limit="${knee_rotation_lower_limit + knee_extension_soft_buffer}"
+                           soft_upper_limit="${knee_rotation_upper_limit - knee_flexion_soft_buffer}"
+                           k_position="${k_position_value_rotary}"
+                           k_velocity="${k_velocity_value_rotary}" />
     </joint>
     <joint name="right_ankle" type="revolute">
@@ -488,6 +548,12 @@
         <origin xyz="0 0 ${-lower_leg_height}" rpy="0 0 0"/>
         <axis xyz="0 1 0"/>
-        <limit velocity="${ankle_velocity_limit}" effort="${ankle_effort_limit}" lower="${ankle_rotation_lower_limit}" upper="${ankle_rotation_upper_limit}"/>
-        <safety_controller soft_lower_limit="${ankle_rotation_lower_limit + ankle_plantarflexion_soft_buffer}" soft_upper_limit="${ankle_rotation_upper_limit - ankle_dorsalflexion_soft_buffer}" k_position="5" k_velocity="${k_velocity_value}" />
+        <limit velocity="${ankle_velocity_limit}"
+               effort="${ankle_effort_limit}"
+               lower="${ankle_rotation_lower_limit}"
+               upper="${ankle_rotation_upper_limit}"/>
+        <safety_controller soft_lower_limit="${ankle_rotation_lower_limit + ankle_plantarflexion_soft_buffer}"
+                           soft_upper_limit="${ankle_rotation_upper_limit - ankle_dorsalflexion_soft_buffer}"
+                           k_position="${k_position_value_linear}"
+                           k_velocity="${k_velocity_value_linear}" />
     </joint>
     <joint name="right_foot_angle" type="fixed">

Commit message: initial commit

File: march_description/urdf/march-iv.xacro (robot description, xacro)
@@ -127,5 +127,4 @@
     </plugin>
     <!-- Used for fixing robot to Gazebo 'base_link' -->
-    <link name="${parent_name}"/>
     <!-- Parts -->
     <!-- Hip-->

Commit message: Fixed the orientation by adding IMU-link in URDF

File: march_description/urdf/march-iv.xacro (robot description, xacro)
@@ -7,4 +7,5 @@
     <!--Important note: when changing value make sure rviz fixed frame is set to the same value (moveit.rviz)-->
     <xacro:property name="parent_name" value="world"/>
+    <xacro:property name="PI" value="3.14159265359"/>
     <xacro:arg name="max_effort_rotary" default="20475" /> <!-- = 25 A -->
     <xacro:arg name="max_effort_linear" default="22932.0" />  <!-- = 28 A -->
@@ -127,4 +128,5 @@
     </plugin>
     <!-- Used for fixing robot to Gazebo 'base_link' -->
+    <link name="${parent_name}"/>
     <!-- Parts -->
     <!-- Hip-->
@@ -155,4 +157,7 @@
         </collision>
     </link>
+    <!-- IMU-->
+    <link name="imu_link">
+    </link>
     <!-- Left Moving Hip-->
     <link name="hip_aa_frame_left_side">
@@ -406,8 +411,12 @@
     </link>
     <!-- Joints -->
+    <joint name="imu_joint" type="fixed">
+        <parent link="${parent_name}"/>
+        <child link="imu_link"/>
+    </joint>
     <joint name="hip" type="fixed">
-        <parent link="${parent_name}"/>
+        <parent link="imu_link"/>
         <child link="hip_base"/>
-        <origin xyz="0 0 ${lower_leg_height+upper_leg_height+hover_height}" rpy="0 0 0"/>
+        <origin xyz="0 0 ${lower_leg_height+upper_leg_height+ankle_plate_height+width/2.0+hover_height}" rpy="0 ${PI/2} 0"/>
     </joint>
     <joint name="left_hip_aa" type="revolute">

Commit message: Fixed the calibration in march_data_collector instead of URDF

File: march_description/urdf/march-iv.xacro (robot description, xacro)
@@ -7,5 +7,4 @@
     <!--Important note: when changing value make sure rviz fixed frame is set to the same value (moveit.rviz)-->
     <xacro:property name="parent_name" value="world"/>
-    <xacro:property name="PI" value="3.14159265359"/>
     <xacro:arg name="max_effort_rotary" default="20475" /> <!-- = 25 A -->
     <xacro:arg name="max_effort_linear" default="22932.0" />  <!-- = 28 A -->
@@ -418,5 +417,5 @@
         <parent link="imu_link"/>
         <child link="hip_base"/>
-        <origin xyz="0 0 ${lower_leg_height+upper_leg_height+ankle_plate_height+width/2.0+hover_height}" rpy="0 ${PI/2} 0"/>
+        <origin xyz="0 0 ${lower_leg_height+upper_leg_height+ankle_plate_height+width/2.0+hover_height}" rpy="0 0 0"/>
     </joint>
     <joint name="left_hip_aa" type="revolute">

Commit message: fixed URDF mistake

File: march_description/urdf/march-iv.xacro (robot description, xacro)
@@ -417,5 +417,5 @@
         <parent link="imu_link"/>
         <child link="hip_base"/>
-        <origin xyz="0 0 ${lower_leg_height+upper_leg_height+ankle_plate_height+width/2.0+hover_height}" rpy="0 0 0"/>
+        <origin xyz="0 0 ${lower_leg_height+upper_leg_height+hover_height}" rpy="0 0 0"/>
     </joint>
     <joint name="left_hip_aa" type="revolute">
