Commit message: Initial structure com_controller plugin

File: march_description/urdf/march4.xacro (robot description, xacro)
@@ -6,6 +6,6 @@
     <!-- Value set to: 'base_link' makes the robot stand on the ground also set launch parameter fixed to false and set
     the hover_height to 0.0-->
-    <xacro:property name="parent_name" value="world"/>
-    <xacro:property name="hover_height" value="0.3"/>
+    <xacro:property name="parent_name" value="base_link"/>
+    <xacro:property name="hover_height" value="0.0"/>
     <xacro:arg name="max_effort_rotary" default="20475" /> <!-- = 25 A -->
     <xacro:arg name="max_effort_linear" default="22932.0" />  <!-- = 28 A -->
@@ -651,5 +651,5 @@
     </transmission>
     <gazebo>
-        <plugin name="model_push" filename="libmodel_push.so"/>
+        <plugin name="com_controller" filename="libcom_controller.so"/>
     </gazebo>
 </robot>

Commit message: Add launch parameter "fixed"

File: march_description/urdf/march4.xacro (robot description, xacro)
@@ -5,6 +5,6 @@
     <!-- Value set to: 'world' fixes the robot to the world-->
     <!-- Value set to: 'base_link' makes the robot stand on the ground-->
-    <xacro:property name="parent_name" value="world"/>
-    <xacro:property name="hover_height" value="0.3"/>
+    <xacro:property name="parent_name" value="base_link"/>
+    <xacro:property name="hover_height" value="0.01"/>
     <xacro:arg name="max_effort_rotary" default="20475" /> <!-- = 25 A -->
     <xacro:arg name="max_effort_linear" default="22932.0" />  <!-- = 28 A -->

Commit message: remove static transformer and change URDF back to old situation

File: march_description/urdf/march4.xacro (robot description, xacro)
@@ -2,7 +2,9 @@
 <!-- Revolute-Revolute Manipulator -->
 <robot name="march" xmlns:xacro="http://www.ros.org/wiki/xacro">
-    <!-- Keep parent_name as base_link for airgaiting/groundgaiting use luanch parameter fixed -->
-    <xacro:property name="parent_name" value="base_link"/>
-    <xacro:property name="hover_height" value="0.01"/>
+    <!-- Switch between airgaiting or standing on the ground-->
+    <!-- Value set to: 'world' fixes the robot to the world-->
+    <!-- Value set to: 'base_link' makes the robot stand on the ground also set launch parameter fixed to false-->
+    <xacro:property name="parent_name" value="world"/>
+    <xacro:property name="hover_height" value="0.3"/>
     <xacro:arg name="max_effort_rotary" default="20475" /> <!-- = 25 A -->
     <xacro:arg name="max_effort_linear" default="22932.0" />  <!-- = 28 A -->

Commit message: Add launch argument for ground gaiting in simulation

File: march_description/urdf/march4.xacro (robot description, xacro)
@@ -6,6 +6,15 @@
     <!-- Value set to: 'base_link' makes the robot stand on the ground also set launch parameter fixed to false and set
     the hover_height to 0.0-->
-    <xacro:property name="parent_name" value="base_link"/>
-    <xacro:property name="hover_height" value="0.0"/>
+    <xacro:unless value="$(arg ground_gait)">
+        <xacro:property name="parent_name" value="world"/>
+        <xacro:property name="hover_height" value="0.3"/>
+    </xacro:unless>
+    <xacro:if value="$(arg ground_gait)">
+        <xacro:property name="parent_name" value="base_link"/>
+        <xacro:property name="hover_height" value="0.0"/>
+        <gazebo>
+            <plugin name="com_controller" filename="libmarch_gazebo_plugins.so"/>
+        </gazebo>
+    </xacro:if>
     <xacro:arg name="max_effort_rotary" default="20475" /> <!-- = 25 A -->
     <xacro:arg name="max_effort_linear" default="22932.0" />  <!-- = 28 A -->
@@ -650,6 +659,3 @@
         </actuator>
     </transmission>
-    <gazebo>
-        <plugin name="com_controller" filename="libmarch_gazebo_plugins.so"/>
-    </gazebo>
 </robot>

Commit message: add multiple K-values

File: march_description/urdf/march4.xacro (robot description, xacro)
@@ -23,12 +23,20 @@
     <xacro:property name="max_effort_linear" value="$(arg max_effort_linear)" />
     <!-- Values for the safety limits, see https://wiki.ros.org/pr2_controller_manager/safety_limits -->
-    <xacro:arg name="k_velocity_value_rotary" default="20000.0" />
-    <xacro:arg name="k_velocity_value_linear" default="20000.0" />
-    <xacro:property name="k_velocity_value_rotary" value="$(arg k_velocity_value_rotary)" />
-    <xacro:property name="k_velocity_value_linear" value="$(arg k_velocity_value_linear)" />
-    <xacro:arg name="k_position_value_rotary" default="5.0" />
-    <xacro:arg name="k_position_value_linear" default="5.0" />
-    <xacro:property name="k_position_value_rotary" value="$(arg k_position_value_rotary)" />
-    <xacro:property name="k_position_value_linear" value="$(arg k_position_value_linear)" />
+    <xacro:arg name="k_velocity_value_hfe" default="20000.0" />
+    <xacro:arg name="k_velocity_value_kfe" default="20000.0" />
+    <xacro:arg name="k_velocity_value_haa" default="20000.0" />
+    <xacro:arg name="k_velocity_value_adpf" default="20000.0" />
+    <xacro:property name="k_velocity_value_hfe" value="$(arg k_velocity_value_hfe)" />
+    <xacro:property name="k_velocity_value_kfe" value="$(arg k_velocity_value_kfe)" />
+    <xacro:property name="k_velocity_value_haa" value="$(arg k_velocity_value_haa)" />
+    <xacro:property name="k_velocity_value_adpf" value="$(arg k_velocity_value_adpf)" />
+    <xacro:arg name="k_position_value_hfe" default="5.0" />
+    <xacro:arg name="k_position_value_kfe" default="5.0" />
+    <xacro:arg name="k_position_value_haa" default="4.0" />
+    <xacro:arg name="k_position_value_adpf" default="4.0" />
+    <xacro:property name="k_position_value_hfe" value="$(arg k_position_value_hfe)" />
+    <xacro:property name="k_position_value_kfe" value="$(arg k_position_value_kfe)" />
+    <xacro:property name="k_position_value_haa" value="$(arg k_position_value_haa)" />
+    <xacro:property name="k_position_value_adpf" value="$(arg k_position_value_adpf)" />
     <!-- Constants for robot dimensions -->
     <!-- Masses determined in https://confluence.projectmarch.nl:8443/display/41TECH/Weights+of+the+Exoskeleton -->
@@ -458,6 +466,6 @@
         <safety_controller soft_lower_limit="${hip_aa_rotation_lower_limit + hip_aa_soft_buffer}"
                            soft_upper_limit="${hip_aa_rotation_upper_limit - hip_aa_soft_buffer}"
-                           k_position="${k_position_value_linear}"
-                           k_velocity="${k_velocity_value_linear}" />
+                           k_position="${k_position_value_haa}"
+                           k_velocity="${k_velocity_value_haa}" />
     </joint>
     <joint name="left_hip_angle" type="fixed">
@@ -477,6 +485,6 @@
         <safety_controller soft_lower_limit="${hip_fe_rotation_lower_limit + hip_fe_soft_buffer}"
                            soft_upper_limit="${hip_fe_rotation_upper_limit - hip_fe_soft_buffer}"
-                           k_position="${k_position_value_rotary}"
-                           k_velocity="${k_velocity_value_rotary}" />
+                           k_position="${k_position_value_hfe}"
+                           k_velocity="${k_velocity_value_hfe}" />
     </joint>
     <joint name="left_knee" type="revolute">
@@ -491,6 +499,6 @@
         <safety_controller soft_lower_limit="${knee_rotation_lower_limit + knee_extension_soft_buffer}"
                            soft_upper_limit="${knee_rotation_upper_limit - knee_flexion_soft_buffer}"
-                           k_position="${k_position_value_rotary}"
-                           k_velocity="${k_velocity_value_rotary}" />
+                           k_position="${k_position_value_kfe}"
+                           k_velocity="${k_velocity_value_kfe}" />
     </joint>
     <joint name="left_ankle" type="revolute">
@@ -505,6 +513,6 @@
         <safety_controller soft_lower_limit="${ankle_rotation_lower_limit + ankle_plantarflexion_soft_buffer}"
                            soft_upper_limit="${ankle_rotation_upper_limit - ankle_dorsalflexion_soft_buffer}"
-                           k_position="${k_position_value_linear}"
-                           k_velocity="${k_velocity_value_linear}" />
+                           k_position="${k_position_value_adpf}"
+                           k_velocity="${k_velocity_value_adpf}" />
     </joint>
     <joint name="left_foot_angle" type="fixed">
@@ -524,6 +532,6 @@
         <safety_controller soft_lower_limit="${hip_aa_rotation_lower_limit + hip_aa_soft_buffer}"
                            soft_upper_limit="${hip_aa_rotation_upper_limit - hip_aa_soft_buffer}"
-                           k_position="${k_position_value_linear}"
-                           k_velocity="${k_velocity_value_linear}" />
+                           k_position="${k_position_value_haa}"
+                           k_velocity="${k_velocity_value_haa}" />
     </joint>
     <joint name="right_hip_angle" type="fixed">
@@ -543,6 +551,6 @@
         <safety_controller soft_lower_limit="${hip_fe_rotation_lower_limit + hip_fe_soft_buffer}"
                            soft_upper_limit="${hip_fe_rotation_upper_limit - hip_fe_soft_buffer}"
-                           k_position="${k_position_value_rotary}"
-                           k_velocity="${k_velocity_value_rotary}" />
+                           k_position="${k_position_value_hfe}"
+                           k_velocity="${k_velocity_value_hfe}" />
     </joint>
     <joint name="right_knee" type="revolute">
@@ -557,6 +565,6 @@
         <safety_controller soft_lower_limit="${knee_rotation_lower_limit + knee_extension_soft_buffer}"
                            soft_upper_limit="${knee_rotation_upper_limit - knee_flexion_soft_buffer}"
-                           k_position="${k_position_value_rotary}"
-                           k_velocity="${k_velocity_value_rotary}" />
+                           k_position="${k_position_value_kfe}"
+                           k_velocity="${k_velocity_value_kfe}" />
     </joint>
     <joint name="right_ankle" type="revolute">
@@ -571,6 +579,6 @@
         <safety_controller soft_lower_limit="${ankle_rotation_lower_limit + ankle_plantarflexion_soft_buffer}"
                            soft_upper_limit="${ankle_rotation_upper_limit - ankle_dorsalflexion_soft_buffer}"
-                           k_position="${k_position_value_linear}"
-                           k_velocity="${k_velocity_value_linear}" />
+                           k_position="${k_position_value_adpf}"
+                           k_velocity="${k_velocity_value_adpf}" />
     </joint>
     <joint name="right_foot_angle" type="fixed">
